Commit message: Ryan R: working implementation of multiple robot spawns. Split up launch and xacro files

File: kinova_description/urdf/drawer.xacro (robot description, xacro)
@@ -113,6 +113,7 @@
     <child link="frame_link" />
     <parent link="${parent}"/>
-<!--    <origin xyz="0 0 0" rpy="0 0 0" /> base z: 0.7425 -->
-    <origin xyz="0.5 0 1.2025" rpy="-1.5708 -3.1416 -1.5708" />
+    <!-- base z: 0.7425 -->
+   <origin xyz="0 0 0" rpy="-1.5708 -3.1416 -1.5708" />
+    <!-- <origin xyz="0.5 0 1.2025" rpy="-1.5708 -3.1416 -1.5708" /> -->
   </joint>
   <transmission name="tran1">

File: kinova_description/urdf/drawer_model.xacro (robot description, xacro)
@@ -13,5 +13,11 @@
     xmlns:physics="http://playerstage.sourceforge.net/gazebo/xmlschema/#physics"
 	xmlns:xacro="http://www.ros.org/wiki/xacro" name="drawer_model">
-  <xacro:include filename="$(find kinova_description)/urdf/drawer.xacro"/>
+  <!-- <xacro:include filename="$(find kinova_description)/urdf/drawer.xacro"/> -->
+  <!-- Don't see a reason to ever need collisin boxes for the drawer. If do, swap xacro with drawer.xacro -->
+  <xacro:arg name="position" default="'0 0 0'" />
+  <xacro:property name="position" value="$(arg position)" />
+  <xacro:arg name="rotation" default="'0 0 0'" />
+  <xacro:property name="rotation" value="$(arg rotation)" />
+  <xacro:include filename="$(find kinova_description)/urdf/drawer_visualization.xacro" />
   <link name="root" />
   <!-- for gazebo -->
@@ -20,6 +26,8 @@
   <joint name="connect_root_and_world" type="fixed">
     <child link="root" />
-    <parent link="world" />
-    <origin xyz="-0.2 0 0" rpy="0 0 0" />
+    <parent link="world" />\
+    <origin xyz="0 0 0" rpy="0 0 0" />
   </joint>
+  <!-- <xacro:property name="robot_root" value="root" />
+  <xacro:drawer  parent="${robot_root}"/> -->
 </robot>

File: kinova_description/urdf/drawer_visualization.xacro (robot description, xacro)
@@ -13,6 +13,6 @@
     xmlns:physics="http://playerstage.sourceforge.net/gazebo/xmlschema/#physics"
 	xmlns:xacro="http://www.ros.org/wiki/xacro">
+  <xacro:macro name="drawer" params="parent position:=^ rotation:=^">
   <xacro:include filename="$(find kinova_description)/urdf/drawer.gazebo" />
-  <xacro:macro name="drawer" params="parent">
   <joint
     name="drawer_slider"
@@ -95,6 +95,7 @@
     <child link="frame_link" />
     <parent link="${parent}"/>
-<!--    <origin xyz="0 0 0" rpy="0 0 0" /> base z: 0.7425 -->
-    <origin xyz="0.5 0 1.2025" rpy="-1.5708 -3.1416 -1.5708" />
+    <!-- base z: 0.7425 -->
+    <origin xyz="${position}" rpy="${rotation}" />
+    <!-- <origin xyz="0.5 0 1.2025" rpy="-1.5708 -3.1416 -1.5708" /> -->
   </joint>
   <transmission name="tran1">

File: kinova_description/urdf/j2s7s300_standalone.xacro (robot description, xacro)
@@ -18,17 +18,11 @@
   <!-- for gazebo -->
   <link name="world"/>
-<!--  <door parent="world"/>-->
-<!--  <link name="cabinet"/>-->
   <joint name="connect_root_and_world" type="fixed">
     <child link="root" />
     <parent link="world" />
-<!--    <origin xyz="-0.2 0.5 0" rpy="0 0 0" /> old yaw: 33.141593  -->
-      <origin xyz="0 0 0.855" rpy="0 0 1.570796" />
+    <origin xyz="1 0 0" rpy="0 0 0" />
+      <!-- <origin xyz="0 0 0.855" rpy="0 0 1.570796" /> -->
+      <!-- <origin xyz="0 0 0" rpy="0 0 0" /> -->
   </joint>
-  <!--  <joint name="door_to_root" type="fixed">-->
-<!--    <child link="cabinet" />-->
-<!--    <parent link="root" />-->
-<!--    <origin xyz="0 0 0" rpy="0 0 0" />-->
-<!--  </joint>-->
   <xacro:property name="robot_root" value="root" />
   <xacro:j2s7s300  base_parent="${robot_root}"/>
