Commit message: Changed to melodic....

File: kinova_gen_3/kortex_description/arms/gen3_lite/6dof/urdf/gen3_lite_macro.xacro (robot description, xacro)
@@ -59,5 +59,5 @@
       <child link="${prefix}shoulder_link" />
       <axis xyz="0 0 1" />
-      <limit lower="-2.68" upper="2.68" effort="10" velocity="1.6" />
+      <limit lower="-2.69" upper="2.69" effort="10" velocity="1.6" />
     </joint>
     <link name="${prefix}arm_link">
@@ -91,5 +91,5 @@
       <child link="${prefix}arm_link" />
       <axis xyz="0 0 1" />
-      <limit lower="-2.61" upper="2.61" effort="14" velocity="1.6" />
+      <limit lower="-2.69" upper="2.69" effort="14" velocity="1.6" />
     </joint>
     <link name="${prefix}forearm_link">
@@ -123,5 +123,5 @@
       <child link="${prefix}forearm_link" />
       <axis xyz="0 0 1" />
-      <limit lower="-2.61" upper="2.61" effort="10" velocity="1.6" />
+      <limit lower="-2.69" upper="2.69" effort="10" velocity="1.6" />
     </joint>
     <link name="${prefix}lower_wrist_link">
@@ -155,5 +155,5 @@
       <child link="${prefix}lower_wrist_link" />
       <axis xyz="0 0 1" />
-      <limit lower="-2.6" upper="2.6" effort="7" velocity="1.6" />
+      <limit lower="-2.59" upper="2.59" effort="7" velocity="1.6" />
     </joint>
     <link name="${prefix}upper_wrist_link">
@@ -187,5 +187,5 @@
       <child link="${prefix}upper_wrist_link" />
       <axis xyz="0 0 1" />
-      <limit lower="-2.53" upper="2.53" effort="7" velocity="1.6" />
+      <limit lower="-2.57" upper="2.57" effort="7" velocity="1.6" />
     </joint>
     <link name="${prefix}end_effector_link"/>
@@ -195,5 +195,5 @@
       <child link="${prefix}end_effector_link" />
       <axis xyz="0 0 1" />
-      <limit lower="-2.6" upper="2.6" effort="7" velocity="3.2" />
+      <limit lower="-2.59" upper="2.59" effort="7" velocity="3.2" />
     </joint>
     <link name="${prefix}dummy_link" />

File: kinova_gen_3/kortex_description/grippers/robotiq_2f_140/urdf/robotiq_2f_140_transmission_macro.xacro (robot description, xacro)
@@ -13,5 +13,5 @@
         </transmission>
         <gazebo>
-            <plugin filename="libroboticsgroup_upatras_gazebo_mimic_joint_plugin.so" name="mimic_robotiq_140_1">
+            <plugin filename="libroboticsgroup_gazebo_mimic_joint_plugin.so" name="mimic_robotiq_140_1">
                 <joint>${prefix}finger_joint</joint>
                 <mimicJoint>${prefix}right_outer_knuckle_joint</mimicJoint>
@@ -21,5 +21,5 @@
                 <hasPID/>
             </plugin>
-            <plugin filename="libroboticsgroup_upatras_gazebo_mimic_joint_plugin.so" name="mimic_robotiq_140_2">
+            <plugin filename="libroboticsgroup_gazebo_mimic_joint_plugin.so" name="mimic_robotiq_140_2">
                 <joint>${prefix}finger_joint</joint>
                 <mimicJoint>${prefix}right_inner_knuckle_joint</mimicJoint>
@@ -29,5 +29,5 @@
                 <hasPID/>
             </plugin>
-            <plugin filename="libroboticsgroup_upatras_gazebo_mimic_joint_plugin.so" name="mimic_robotiq_140_3">
+            <plugin filename="libroboticsgroup_gazebo_mimic_joint_plugin.so" name="mimic_robotiq_140_3">
                 <joint>${prefix}finger_joint</joint>
                 <mimicJoint>${prefix}left_inner_knuckle_joint</mimicJoint>
@@ -37,5 +37,5 @@
                 <hasPID/>
             </plugin>
-            <plugin filename="libroboticsgroup_upatras_gazebo_mimic_joint_plugin.so" name="mimic_robotiq_140_4">
+            <plugin filename="libroboticsgroup_gazebo_mimic_joint_plugin.so" name="mimic_robotiq_140_4">
                 <joint>${prefix}finger_joint</joint>
                 <mimicJoint>${prefix}left_inner_finger_joint</mimicJoint>
@@ -45,5 +45,5 @@
                 <hasPID/>
             </plugin>
-            <plugin filename="libroboticsgroup_upatras_gazebo_mimic_joint_plugin.so" name="mimic_robotiq_140_5">
+            <plugin filename="libroboticsgroup_gazebo_mimic_joint_plugin.so" name="mimic_robotiq_140_5">
                 <joint>${prefix}finger_joint</joint>
                 <mimicJoint>${prefix}right_inner_finger_joint</mimicJoint>

File: kinova_gen_3/kortex_description/grippers/robotiq_2f_85/urdf/robotiq_2f_85_transmission_macro.xacro (robot description, xacro)
@@ -13,5 +13,5 @@
         </transmission>
         <gazebo>
-            <plugin filename="libroboticsgroup_upatras_gazebo_mimic_joint_plugin.so" name="mimic_robotiq_85_1">
+            <plugin filename="libroboticsgroup_gazebo_mimic_joint_plugin.so" name="mimic_robotiq_85_1">
                 <joint>${prefix}finger_joint</joint>
                 <mimicJoint>${prefix}right_outer_knuckle_joint</mimicJoint>
@@ -21,5 +21,5 @@
                 <hasPID/>
             </plugin>
-            <plugin filename="libroboticsgroup_upatras_gazebo_mimic_joint_plugin.so" name="mimic_robotiq_85_2">
+            <plugin filename="libroboticsgroup_gazebo_mimic_joint_plugin.so" name="mimic_robotiq_85_2">
                 <joint>${prefix}finger_joint</joint>
                 <mimicJoint>${prefix}right_inner_knuckle_joint</mimicJoint>
@@ -29,5 +29,5 @@
                 <hasPID/>
             </plugin>
-            <plugin filename="libroboticsgroup_upatras_gazebo_mimic_joint_plugin.so" name="mimic_robotiq_85_3">
+            <plugin filename="libroboticsgroup_gazebo_mimic_joint_plugin.so" name="mimic_robotiq_85_3">
                 <joint>${prefix}finger_joint</joint>
                 <mimicJoint>${prefix}left_inner_knuckle_joint</mimicJoint>
@@ -37,5 +37,5 @@
                 <hasPID/>
             </plugin>
-            <plugin filename="libroboticsgroup_upatras_gazebo_mimic_joint_plugin.so" name="mimic_robotiq_85_4">
+            <plugin filename="libroboticsgroup_gazebo_mimic_joint_plugin.so" name="mimic_robotiq_85_4">
                 <joint>${prefix}finger_joint</joint>
                 <mimicJoint>${prefix}left_inner_finger_joint</mimicJoint>
@@ -45,5 +45,5 @@
                 <hasPID/>
             </plugin>
-            <plugin filename="libroboticsgroup_upatras_gazebo_mimic_joint_plugin.so" name="mimic_robotiq_85_5">
+            <plugin filename="libroboticsgroup_gazebo_mimic_joint_plugin.so" name="mimic_robotiq_85_5">
                 <joint>${prefix}finger_joint</joint>
                 <mimicJoint>${prefix}right_inner_finger_joint</mimicJoint>
